File: hardware/kicad/accumelator.sch (KiCad schematic (older format))
At the start: 10 parts, among them U1 74LS04

Commit message: Just a backup.
Parts:
- removed C0: 100nF, Capacitors_THT:C_Disc_D5.0mm_W2.5mm_P2.50mm, symbol C
- removed U1: 74LS04, Housings_DIP:DIP-14_W7.62mm, symbol 74LS04
- C10, C11, C7, C9: footprint Capacitors_THT:C_Disc_D5.0mm_W2.5mm_P2.50mm -> Capacitors_ThroughHole:C_Disc_D3_P2.5
Connections:
- net Ctrl_ACC_Source: now also ACC_Data_In_Buffer1.19 (CE)
- net GND: now also C9.2; no longer C9.1
- net VCC: now also C9.1; no longer C9.2
Other:
- moved on the sheet: C7, C9
Changed lines of the file:
@@
 LIBS:switches
 LIBS:relays
-LIBS:motors
 LIBS:transistors
 LIBS:conn
@@
 LIBS:valves
 LIBS:at28hcXXX
-LIBS:amm816-cache
+LIBS:main-cache
 EELAYER 25 0
 EELAYER END
 $Descr A4 11693 8268
 encoding utf-8
-Sheet 2 7
-Title "AMM816 - Accumelator"
+Sheet 2 6
+Title "AMM812 - Accumelator"
 Date ""
 Rev ""
@@
 $EndComp
 $Comp
-L 74LS04 U1
-U 1 1 5A0C410A
-P 1400 3400
-F 0 "U1" H 1595 3515 50  0000 C CNN
-F 1 "74LS04" H 1590 3275 50  0000 C CNN
-F 2 "Housings_DIP:DIP-14_W7.62mm" H 1400 3400 50  0001 C CNN
-F 3 "" H 1400 3400 50  0001 C CNN
-	1    1400 3400
-	0    -1   -1   0
-$EndComp
-$Comp
 L GND #PWR08
 U 1 1 5A0C410B
@@
 Text GLabel 5400 2350 1    60   Input ~ 0
 Ctrl_ACC_Output
-Text GLabel 1400 6350 3    60   Input ~ 0
+Text GLabel 1450 2650 0    60   Input ~ 0
 Ctrl_ACC_Source
 Text GLabel 5250 6350 3    60   Input ~ 0
@@
 Text HLabel 8800 5650 3    60   Output ~ 0
 ALU_A[0..7]
-Text GLabel 1350 2250 0    60   BiDi ~ 0
+Text GLabel 1400 2250 0    60   3State ~ 0
 Data[0..7]
 Text HLabel 2450 4150 0    60   Input ~ 0
@@
 $EndComp
 $Comp
-L C C0
-U 1 1 5A0F4C4B
-P 2050 3250
-F 0 "C0" H 2075 3350 50  0000 L CNN
-F 1 "100nF" H 2075 3150 50  0000 L CNN
-F 2 "Capacitors_THT:C_Disc_D5.0mm_W2.5mm_P2.50mm" H 2088 3100 50  0001 C CNN
-F 3 "" H 2050 3250 50  0001 C CNN
-	1    2050 3250
-	1    0    0    -1
-$EndComp
-$Comp
-L VCC #PWR011
-U 1 1 5A0F4EFF
-P 2050 3100
-F 0 "#PWR011" H 2050 2950 50  0001 C CNN
-F 1 "VCC" H 2050 3250 50  0000 C CNN
-F 2 "" H 2050 3100 50  0001 C CNN
-F 3 "" H 2050 3100 50  0001 C CNN
-	1    2050 3100
-	1    0    0    -1
-$EndComp
-$Comp
 L C C11
 U 1 1 5A0F6050
@@
 F 0 "C11" H 8025 6050 50  0000 L CNN
 F 1 "100nF" H 8025 5850 50  0000 L CNN
-F 2 "Capacitors_THT:C_Disc_D5.0mm_W2.5mm_P2.50mm" H 8038 5800 50  0001 C CNN
+F 2 "Capacitors_ThroughHole:C_Disc_D3_P2.5" H 8038 5800 50  0001 C CNN
 F 3 "" H 8000 5950 50  0001 C CNN
 	1    8000 5950
@@
 F 0 "C10" H 8025 4250 50  0000 L CNN
 F 1 "100nF" H 8025 4050 50  0000 L CNN
-F 2 "Capacitors_THT:C_Disc_D5.0mm_W2.5mm_P2.50mm" H 8038 4000 50  0001 C CNN
+F 2 "Capacitors_ThroughHole:C_Disc_D3_P2.5" H 8038 4000 50  0001 C CNN
 F 3 "" H 8000 4150 50  0001 C CNN
 	1    8000 4150
@@
 L C C9
 U 1 1 5A0F6391
-P 8000 2700
-F 0 "C9" H 8025 2800 50  0000 L CNN
-F 1 "100nF" H 8025 2600 50  0000 L CNN
-F 2 "Capacitors_THT:C_Disc_D5.0mm_W2.5mm_P2.50mm" H 8038 2550 50  0001 C CNN
-F 3 "" H 8000 2700 50  0001 C CNN
-	1    8000 2700
-	-1   0    0    1
+P 8100 2700
+F 0 "C9" H 8125 2800 50  0000 L CNN
+F 1 "100nF" H 8125 2600 50  0000 L CNN
+F 2 "Capacitors_ThroughHole:C_Disc_D3_P2.5" H 8138 2550 50  0001 C CNN
+F 3 "" H 8100 2700 50  0001 C CNN
+	1    8100 2700
+	0    -1   -1   0
 $EndComp
 $Comp
 L C C7
 U 1 1 5A0F63E6
-P 3550 1400
-F 0 "C7" H 3575 1500 50  0000 L CNN
-F 1 "100nF" H 3575 1300 50  0000 L CNN
-F 2 "Capacitors_THT:C_Disc_D5.0mm_W2.5mm_P2.50mm" H 3588 1250 50  0001 C CNN
-F 3 "" H 3550 1400 50  0001 C CNN
-	1    3550 1400
+P 3200 1350
+F 0 "C7" H 3225 1450 50  0000 L CNN
+F 1 "100nF" H 3225 1250 50  0000 L CNN
+F 2 "Capacitors_ThroughHole:C_Disc_D3_P2.5" H 3238 1200 50  0001 C CNN
+F 3 "" H 3200 1350 50  0001 C CNN
+	1    3200 1350
 	0    -1   -1   0
 $EndComp
 $Comp
+L GND #PWR011
+U 1 1 5A0F7405
+P 8000 6100
+F 0 "#PWR011" H 8000 5850 50  0001 C CNN
+F 1 "GND" H 8000 5950 50  0000 C CNN
+F 2 "" H 8000 6100 50  0001 C CNN
+F 3 "" H 8000 6100 50  0001 C CNN
+	1    8000 6100
+	1    0    0    -1
+$EndComp
+$Comp
 L GND #PWR012
-U 1 1 5A0F7405
-P 8000 6300
-F 0 "#PWR012" H 8000 6050 50  0001 C CNN
-F 1 "GND" H 8000 6150 50  0000 C CNN
-F 2 "" H 8000 6300 50  0001 C CNN
-F 3 "" H 8000 6300 50  0001 C CNN
-	1    8000 6300
+U 1 1 5A0F7559
+P 8000 4300
+F 0 "#PWR012" H 8000 4050 50  0001 C CNN
+F 1 "GND" H 8000 4150 50  0000 C CNN
+F 2 "" H 8000 4300 50  0001 C CNN
+F 3 "" H 8000 4300 50  0001 C CNN
+	1    8000 4300
 	1    0    0    -1
 $EndComp
 $Comp
 L GND #PWR013
-U 1 1 5A0F7559
-P 8000 4500
-F 0 "#PWR013" H 8000 4250 50  0001 C CNN
-F 1 "GND" H 8000 4350 50  0000 C CNN
-F 2 "" H 8000 4500 50  0001 C CNN
-F 3 "" H 8000 4500 50  0001 C CNN
-	1    8000 4500
-	1    0    0    -1
+U 1 1 5A0F7876
+P 8250 2700
+F 0 "#PWR013" H 8250 2450 50  0001 C CNN
+F 1 "GND" H 8250 2550 50  0000 C CNN
+F 2 "" H 8250 2700 50  0001 C CNN
+F 3 "" H 8250 2700 50  0001 C CNN
+	1    8250 2700
+	0    -1   -1   0
 $EndComp
 $Comp
 L GND #PWR014
-U 1 1 5A0F7876
-P 8250 2850
-F 0 "#PWR014" H 8250 2600 50  0001 C CNN
-F 1 "GND" H 8250 2700 50  0000 C CNN
-F 2 "" H 8250 2850 50  0001 C CNN
-F 3 "" H 8250 2850 50  0001 C CNN
-	1    8250 2850
+U 1 1 5A0F7A04
+P 3350 1350
+F 0 "#PWR014" H 3350 1100 50  0001 C CNN
+F 1 "GND" H 3350 1200 50  0000 C CNN
+F 2 "" H 3350 1350 50  0001 C CNN
+F 3 "" H 3350 1350 50  0001 C CNN
+	1    3350 1350
 	0    -1   -1   0
 $EndComp
 $Comp
-L GND #PWR015
-U 1 1 5A0F7A04
-P 3700 1400
-F 0 "#PWR015" H 3700 1150 50  0001 C CNN
-F 1 "GND" H 3700 1250 50  0000 C CNN
-F 2 "" H 3700 1400 50  0001 C CNN
-F 3 "" H 3700 1400 50  0001 C CNN
-	1    3700 1400
+L VCC #PWR015
+U 1 1 5A0F7A5D
+P 3050 1350
+F 0 "#PWR015" H 3050 1200 50  0001 C CNN
+F 1 "VCC" H 3050 1500 50  0000 C CNN
+F 2 "" H 3050 1350 50  0001 C CNN
+F 3 "" H 3050 1350 50  0001 C CNN
+	1    3050 1350
 	0    -1   -1   0
 $EndComp
 $Comp
 L VCC #PWR016
-U 1 1 5A0F7A5D
-P 3200 1300
-F 0 "#PWR016" H 3200 1150 50  0001 C CNN
-F 1 "VCC" H 3200 1450 50  0000 C CNN
-F 2 "" H 3200 1300 50  0001 C CNN
-F 3 "" H 3200 1300 50  0001 C CNN
-	1    3200 1300
-	1    0    0    -1
+U 1 1 5A0F7ABA
+P 7950 2700
+F 0 "#PWR016" H 7950 2550 50  0001 C CNN
+F 1 "VCC" H 7950 2850 50  0000 C CNN
+F 2 "" H 7950 2700 50  0001 C CNN
+F 3 "" H 7950 2700 50  0001 C CNN
+	1    7950 2700
+	0    -1   -1   0
 $EndComp
 $Comp
 L VCC #PWR017
-U 1 1 5A0F7ABA
-P 8000 2550
-F 0 "#PWR017" H 8000 2400 50  0001 C CNN
-F 1 "VCC" H 8000 2700 50  0000 C CNN
-F 2 "" H 8000 2550 50  0001 C CNN
-F 3 "" H 8000 2550 50  0001 C CNN
-	1    8000 2550
-	1    0    0    -1
-$EndComp
-$Comp
-L VCC #PWR018
 U 1 1 5A0F7AE9
 P 8000 4000
-F 0 "#PWR018" H 8000 3850 50  0001 C CNN
+F 0 "#PWR017" H 8000 3850 50  0001 C CNN
 F 1 "VCC" H 8000 4150 50  0000 C CNN
 F 2 "" H 8000 4000 50  0001 C CNN
@@
 $EndComp
 $Comp
-L VCC #PWR019
+L VCC #PWR018
 U 1 1 5A0F7BC9
 P 8000 5800
-F 0 "#PWR019" H 8000 5650 50  0001 C CNN
+F 0 "#PWR018" H 8000 5650 50  0001 C CNN
 F 1 "VCC" H 8000 5950 50  0000 C CNN
 F 2 "" H 8000 5800 50  0001 C CNN
@@
 	6500 3700 6500 3600
 Wire Wire Line
-	1400 3850 1400 6350
-Wire Wire Line
 	6250 5500 6500 5500
 Wire Wire Line
@@
 	5400 2550 6500 2550
 Wire Wire Line
-	1400 2650 2500 2650
-Wire Wire Line
-	1400 2650 1400 2950
+	1450 2650 2500 2650
 Wire Wire Line
 	6500 3950 5600 3950
@@
 	5900 950  1700 950
 Wire Bus Line
-	1700 2250 1350 2250
+	1700 2250 1400 2250
 Connection ~ 6500 3700
 Connection ~ 6500 5750
@@
 Wire Wire Line
 	1950 2550 2500 2550
-Wire Wire Line
-	1500 3450 2300 3450
-Wire Wire Line
-	2050 3450 2050 3400
-Connection ~ 2050 3450
-Wire Wire Line
-	3400 1400 3200 1400
-Wire Wire Line
-	3200 1300 3200 1600
-Connection ~ 3200 1400
-Wire Wire Line
-	7200 2600 7200 2850
-Wire Wire Line
-	7200 2850 8250 2850
-Wire Wire Line
-	8000 4300 8000 4500
-Wire Wire Line
-	8000 4450 6900 4450
-Wire Wire Line
-	6900 4450 6900 4300
-Wire Wire Line
-	8000 6100 8000 6300
-Wire Wire Line
-	8000 6250 6900 6250
-Wire Wire Line
-	6900 6250 6900 6100
-Connection ~ 8000 6250
-Connection ~ 8000 4450
 Wire Bus Line
-	3150 5150 3150 4150
+	3150 4150 3150 5150
 Wire Bus Line
 	3150 4150 2450 4150
-$Comp
-L GND #PWR020
-U 1 1 5A0F4EBC
-P 2300 3450
-F 0 "#PWR020" H 2300 3200 50  0001 C CNN
-F 1 "GND" H 2300 3300 50  0000 C CNN
-F 2 "" H 2300 3450 50  0001 C CNN
-F 3 "" H 2300 3450 50  0001 C CNN
-	1    2300 3450
-	0    -1   -1   0
-$EndComp
-Connection ~ 8000 2850
 $EndSCHEMATC

Commit message: Just a backup.
Parts:
- removed ACC_High1, ACC_Low1: 74LS173, Housings_DIP:DIP-16_W7.62mm, symbol 74LS173
- removed C10, C11: 100nF, Capacitors_ThroughHole:C_Disc_D3_P2.5, symbol C
- added Register_Bus1: CONN_02X13, Pin_Headers:Pin_Header_Straight_2x13_Pitch2.00mm, symbol CONN_02X13
- added U3: 74LS04, Housings_DIP:DIP-14_W7.62mm, symbol 74LS04
Connections:
- net ALU_A0: now also Register_Bus1.2 (P2)
- net ALU_A1: now also Register_Bus1.4 (P4)
- net ALU_A2: now also Register_Bus1.6 (P6)
- net ALU_A3: now also Register_Bus1.8 (P8)
- net ALU_A4: now also Register_Bus1.10 (P10)
- net ALU_A5: now also Register_Bus1.12 (P12)
- net ALU_A6: now also Register_Bus1.14 (P14)
- net ALU_A7: now also Register_Bus1.16 (P16)
- net ALU_Output0: now also Register_Bus1.1 (P1)
- net ALU_Output1: now also Register_Bus1.3 (P3)
- net ALU_Output2: now also Register_Bus1.5 (P5)
- net ALU_Output3: now also Register_Bus1.7 (P7)
- net ALU_Output4: now also Register_Bus1.9 (P9)
- net ALU_Output5: now also Register_Bus1.11 (P11)
- net ALU_Output6: now also Register_Bus1.13 (P13)
- net ALU_Output7: now also Register_Bus1.15 (P15)
- net Clock: now also Register_Bus1.20 (P20)
- net GND: now also Register_Bus1.24 (P24), Register_Bus1.26 (P26), U3.7 (GND)
- net Reset: now also Register_Bus1.18 (P18)
- net VCC: now also Register_Bus1.25 (P25), U3.14 (VCC)
- net Ctrl_ACC_Output renamed Ctrl_ACC_Output_I
- net Ctrl_ACC_Source: no longer names the net of ACC_Data_In_Buffer1.19 (CE)
- net Ctrl_ACC_Source: now also U3.2
- new net Ctrl_ACC_Input_I: Register_Bus1.22 (P22)
- new net Ctrl_ALU_Enable_I: U3.1
- new net Register0: Register_Bus1.17 (P17)
- new net Register1: Register_Bus1.19 (P19)
- new net Register2: Register_Bus1.21 (P21)
- new net Register3: Register_Bus1.23 (P23)
Other:
- moved on the sheet: C9
