File: hardware/kicad/alu.sch (KiCad schematic (older format))
At the start: 11 parts, among them U1 74LS04, U9 74LS08

Commit message: Just a backup.
Parts:
- removed C3, C6: 100nF, Capacitors_THT:C_Disc_D5.0mm_W2.5mm_P2.50mm, symbol C
- removed Sys_Flags1: 74LS173, Housings_DIP:DIP-16_W7.62mm, symbol 74LS173
- removed U1: 74LS04, Housings_DIP:DIP-14_W7.62mm, symbol 74LS04
- removed U9: 74LS08, Housings_DIP:DIP-14_W7.62mm, symbol 74LS08
- C2, C4, C5: footprint Capacitors_THT:C_Disc_D5.0mm_W2.5mm_P2.50mm -> Capacitors_ThroughHole:C_Disc_D3_P2.5
- renumbered Usr_Flags1 to Flags1
Connections:
- net labels added: IR[0..3]
- net labels removed: Ctrl_Select_Flags, IR3, IR[0..7]
- wire segments 128 -> 94
- no-connect marks 5 -> 3
Other:
- moved on the sheet: C4, C5

Commit message: Just a backup.
Connections:
- net GND: no longer ALU_Low1.24 (A10), ALU_Low1.28 (A9)
- net VCC: no longer ALU_High1.23 (CE), ALU_High1.31 (WE), ALU_Low1.23 (CE), ALU_Low1.31 (WE)
- net Ctrl_ALU_Enable renamed Ctrl_ALU_Enable_I
- net Ctrl_ALU_Enable_I: now also ALU_High1.23 (CE), ALU_High1.31 (WE), ALU_Low1.23 (CE), ALU_Low1.24 (A10), ALU_Low1.28 (A9), ALU_Low1.31 (WE)
