File: hardware/kicad/ir.sch (KiCad schematic (older format))
At the start: 8 parts

Commit message: Just a backup.
Parts:
- added C10: 100nF, Capacitors_ThroughHole:C_Disc_D3_P2.5, symbol C_Small
- added IR_High1: 74LS173, Housings_DIP:DIP-16_W7.62mm, symbol 74LS173
- added U3: 74LS04, symbol 74LS04
- added U4: 74LS245, Housings_DIP:DIP-20_W7.62mm, symbol 74LS245
- renumbered IR1 to IR_Low1
Connections:
- net Clock: now also IR_High1.7 (Cp)
- net Data0: now also MAR_A1.14 (D0), MAR_C1.14 (D0), U4.2 (A0); no longer MAR_B1.14 (D0)
- net Data1: now also MAR_A1.13 (D1), MAR_C1.13 (D1), U4.3 (A1); no longer MAR_B1.13 (D1)
- net Data2: now also MAR_A1.12 (D2), MAR_C1.12 (D2), U4.4 (A2); no longer MAR_B1.12 (D2)
- net Data3: now also MAR_A1.11 (D3), MAR_C1.11 (D3), U4.5 (A3); no longer MAR_B1.11 (D3)
- net Data4: now also MAR_B1.14 (D0), IR_High1.14 (D0); no longer MAR_A1.14 (D0), MAR_C1.14 (D0)
- net Data5: now also MAR_B1.13 (D1), IR_High1.13 (D1); no longer MAR_A1.13 (D1), MAR_C1.13 (D1)
- net Data6: now also MAR_B1.12 (D2), IR_High1.12 (D2); no longer MAR_A1.12 (D2), MAR_C1.12 (D2)
- net Data7: now also MAR_B1.11 (D3), IR_High1.11 (D3); no longer MAR_A1.11 (D3), MAR_C1.11 (D3)
- net GND: now also C10.2, IR_High1.8 (GND), U3.7 (GND), U4.10 (GND), U4.6 (A4), U4.7 (A5), U4.8 (A6), U4.9 (A7)
- net IR0: now also U4.18 (B0)
- net IR1: now also U4.17 (B1)
- net IR2: now also U4.16 (B2)
- net IR3: now also U4.15 (B3)
- net Reset: now also IR_High1.15 (Mr)
- net VCC: now also C10.1, IR_High1.16 (VCC), U3.14 (VCC), U4.1 (A->B), U4.20 (VCC); no longer IR_Low1.1 (Oe1), IR_Low1.2 (Oe2)
- net Ctrl_MAR_High_Input renamed Ctrl_MAR_High_Input_I
- net Ctrl_MAR_High_Input_I: no longer MAR_B1.10 (E2), MAR_B1.9 (E1)
- net Ctrl_MAR_Low_Input renamed Ctrl_IR_Input_I
- net Ctrl_IR_Input_I: now also IR_High1.10 (E2), IR_High1.9 (E1), U3.5, U4.19 (CE); no longer MAR_A1.10 (E2), MAR_A1.9 (E1)
- net Ctrl_MAR_Output renamed Ctrl_MAR_Output_I
- new net: IR_High1.1 (Oe1), IR_High1.2 (Oe2), IR_Low1.1 (Oe1), IR_Low1.2 (Oe2), U3.6
- new net Ctrl_MAR_Low_Input_I: MAR_A1.10 (E2), MAR_A1.9 (E1), MAR_B1.10 (E2), MAR_B1.9 (E1)
- new net Register0: IR_High1.3 (Q0)
- new net Register1: IR_High1.4 (Q1)
- new net Register2: IR_High1.5 (Q2)
- new net Register3: IR_High1.6 (Q3)
- no-connect marks 0 -> 4
Other:
- moved on the sheet: C15, C16, C17, C18, IR_Low1, MAR_A1, MAR_B1, MAR_C1
