File: hardware/kicad/main.sch (KiCad schematic (older format))
At the start: 7 parts, among them U9 74LS08

Commit message: Just a backup.
Parts:
- removed C39, C40: 100uF, Capacitors_THT:CP_Radial_D5.0mm_P2.50mm, symbol CP1
- removed Power1, Reset_and_Clock1: Conn_01x02_Male, Connectors_Molex:Molex_KK-6410-02_02x2.54mm_Straight, symbol Conn_01x02_Male
- removed System_Bus1: Conn_02x20_Top_Bottom, Pin_Headers:Pin_Header_Straight_2x20_Pitch2.54mm, symbol Conn_02x20_Top_Bottom
- removed U9: 74LS08, Housings_DIP:DIP-14_W7.62mm, symbol 74LS08
- added P1: CONN_02X20, Socket_Strips:Socket_Strip_Straight_2x20, symbol CONN_02X20
- added Power1: CONN_01X02, Connectors_Molex:Molex_KK-6410-02_02x2.54mm_Straight, symbol CONN_01X02
- C1: footprint Capacitors_THT:CP_Radial_D5.0mm_P2.50mm -> Capacitors_ThroughHole:C_Radial_D7.5_L11.2_P2.5
Connections:
- net labels added: Address[0..11], DMA
- net labels removed: Acknowledge, Address12, Address13, Address14, Address15, Address[0..15], Halt, IR6, IR7, IR[0..7], Interrupt
- wire segments 69 -> 44
Other:
- moved on the sheet: C1

Commit message: Just a backup.
Parts:
- C1: footprint Capacitors_ThroughHole:C_Radial_D7.5_L11.2_P2.5 -> Capacitors_ThroughHole:C_Radial_D5_L11_P2.5
- System_Bus1: renamed from P1; footprint Socket_Strips:Socket_Strip_Straight_2x20 -> Pin_Headers:Pin_Header_Straight_2x20_Pitch2.00mm
Changed lines of the file:
@@
 ALU_Output[0..7]
 $Comp
-L GND #PWR01
+L GND #PWR4
 U 1 1 5A0E47E9
 P 4250 5450
-F 0 "#PWR01" H 4250 5200 50  0001 C CNN
+F 0 "#PWR4" H 4250 5200 50  0001 C CNN
 F 1 "GND" H 4250 5300 50  0000 C CNN
 F 2 "" H 4250 5450 50  0001 C CNN
@@
 F 0 "C1" H 3975 5350 50  0000 L CNN
 F 1 "100uF" H 3975 5150 50  0000 L CNN
-F 2 "Capacitors_ThroughHole:C_Radial_D7.5_L11.2_P2.5" H 3950 5250 50  0001 C CNN
+F 2 "Capacitors_ThroughHole:C_Radial_D5_L11_P2.5" H 3950 5250 50  0001 C CNN
 F 3 "" H 3950 5250 50  0001 C CNN
 	1    3950 5250
@@
 Address[0..11]
 $Comp
-L VCC #PWR02
+L VCC #PWR3
 U 1 1 5A16B699
 P 4250 5050
-F 0 "#PWR02" H 4250 4900 50  0001 C CNN
+F 0 "#PWR3" H 4250 4900 50  0001 C CNN
 F 1 "VCC" H 4250 5200 50  0000 C CNN
 F 2 "" H 4250 5050 50  0001 C CNN
@@
 $EndSheet
 $Comp
-L GND #PWR03
+L GND #PWR1
 U 1 1 5A1A56FA
 P 3500 3600
-F 0 "#PWR03" H 3500 3350 50  0001 C CNN
+F 0 "#PWR1" H 3500 3350 50  0001 C CNN
 F 1 "GND" H 3500 3450 50  0000 C CNN
 F 2 "" H 3500 3600 50  0001 C CNN
@@
 $EndComp
 $Comp
-L VCC #PWR04
+L VCC #PWR2
 U 1 1 5A1A5732
 P 3500 3800
-F 0 "#PWR04" H 3500 3650 50  0001 C CNN
+F 0 "#PWR2" H 3500 3650 50  0001 C CNN
 F 1 "VCC" H 3500 3950 50  0000 C CNN
 F 2 "" H 3500 3800 50  0001 C CNN
@@
 Address[0..11]
 $Comp
-L CONN_02X20 P1
+L CONN_02X20 System_Bus1
 U 1 1 5BB52184
 P 3050 2850
-F 0 "P1" H 3050 3900 50  0000 C CNN
+F 0 "System_Bus1" H 3050 3900 50  0000 C CNN
 F 1 "CONN_02X20" V 3050 2850 50  0000 C CNN
-F 2 "Socket_Strips:Socket_Strip_Straight_2x20" H 3050 1900 50  0001 C CNN
+F 2 "Pin_Headers:Pin_Header_Straight_2x20_Pitch2.00mm" H 3050 1900 50  0001 C CNN
 F 3 "" H 3050 1900 50  0000 C CNN
 	1    3050 2850
@@
 Connection ~ 3300 2500
 $Comp
-L PWR_FLAG #FLG05
+L PWR_FLAG #FLG1
 U 1 1 5A0F12B3
 P 3700 4800
-F 0 "#FLG05" H 3700 4875 50  0001 C CNN
+F 0 "#FLG1" H 3700 4875 50  0001 C CNN
 F 1 "PWR_FLAG" H 3700 4950 50  0000 C CNN
 F 2 "" H 3700 4800 50  0001 C CNN
@@
 $EndComp
 $Comp
-L PWR_FLAG #FLG06
+L PWR_FLAG #FLG2
 U 1 1 5A0F2A42
 P 3700 5900
-F 0 "#FLG06" H 3700 5975 50  0001 C CNN
+F 0 "#FLG2" H 3700 5975 50  0001 C CNN
 F 1 "PWR_FLAG" H 3700 6050 50  0000 C CNN
 F 2 "" H 3700 5900 50  0001 C CNN
