File: hardware/kicad/main.kicad_pcb (KiCad board)
At the start: 2 copper layers, 150 x 100 mm, 43 parts, among them P1 CONN_02X20, U1 74LS245, U2 74LS245

Commit message: Just a backup.
Parts:
- removed ACC_High1, ACC_Low1, IR1: 74LS173, Housings_DIP:DIP-16_W7.62mm
- removed C14, C33: 100nF, Capacitors_ThroughHole:C_Disc_D3_P2.5
- removed Decode_A1, Decode_B1: AT28HC64BF, PLCC32_bugfix:PLCC-32_THT-Socket_bugfix
- removed P1: CONN_02X20, Socket_Strips:Socket_Strip_Straight_2x20
- added Decode1: AT28HC64BF, PLCC32_bugfix:PLCC-32_THT-Socket_bugfix, F.Cu at (195.0, 102.5)
- added G***: LOGO, Logo:logo, F.Cu at (177.5, 130.0)
- added IR_High1: 74LS173, Housings_DIP:DIP-16_W7.62mm, F.Cu at (110.0, 97.5)
- added IR_Low1: 74LS173, Housings_DIP:DIP-16_W7.62mm, F.Cu at (167.5, 100.0)
- added REF1: 1pin, Connect:1pin, F.Cu at (67.5, 67.5)
- added REF2: 1pin, Connect:1pin, F.Cu at (202.5, 67.5)
- added REF3: 1pin, Connect:1pin, F.Cu at (202.5, 152.5)
- added REF4: 1pin, Connect:1pin, F.Cu at (67.5, 152.5)
- added Register_Bus1: CONN_02X13, Pin_Headers:Pin_Header_Straight_2x13_Pitch2.00mm, F.Cu at (95.0, 67.5)
- added System_Bus1: CONN_02X20, Pin_Headers:Pin_Header_Straight_2x20_Pitch2.00mm, F.Cu at (92.5, 152.5)
- added U3: 74LS04, Housings_DIP:DIP-14_W7.62mm, F.Cu at (87.5, 140.0)
- added U4: 74LS245, Housings_DIP:DIP-20_W7.62mm, F.Cu at (155.0, 67.5)
- C1: footprint Capacitors_ThroughHole:C_Radial_D7.5_L11.2_P2.5 -> Capacitors_ThroughHole:C_Radial_D5_L11_P2.5
- moved C7 71.6 mm to (160.0, 95.0)
- moved C13 54.9 mm to (67.5, 142.5), turned to 270 degrees
- moved U1 30.4 mm to (130.0, 120.0)
- moved C2 28.5 mm to (115.0, 120.0), turned to 180 degrees
- moved PC_B1 20.2 mm to (120.0, 87.5)
- moved ACC_Output_Buffer1 15.0 mm to (92.5, 102.5)
- moved C6 15.0 mm to (95.0, 130.0)
- moved PC_C1 15.0 mm to (130.0, 105.0)
- moved C10 11.2 mm to (142.5, 82.5), turned to 270 degrees
- moved Lookup1 10.6 mm to (195.0, 77.5)
- moved C11 10.3 mm to (142.5, 70.0), turned to 270 degrees
- moved PC_A1 10.0 mm to (120.0, 75.0)
- moved C17 7.91 mm to (172.5, 92.5)
- moved T_Stage1 7.91 mm to (170.0, 70.0)
- moved ALU_Low1 5.59 mm to (77.5, 120.0)
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Connections:
- net Ctrl_MAR_Output renamed Ctrl_MAR_Output_I
- ACC_Data_In_Buffer1 pad 19: Ctrl_ACC_Source -> Net-(ACC_Data_In_Buffer1-Pad19)
- ACC_Output_Buffer1 pad 19: Ctrl_ACC_Output -> Ctrl_ACC_Output_I
- ALU_High1 pad 23: VCC -> Ctrl_ALU_Enable_I
- ALU_High1 pad 25: Ctrl_ALU_Enable -> Ctrl_ALU_Enable_I
- ALU_High1 pad 31: VCC -> Ctrl_ALU_Enable_I
- ALU_Low1 pad 23: VCC -> Ctrl_ALU_Enable_I
- ALU_Low1 pad 24: GND -> Ctrl_ALU_Enable_I
- ALU_Low1 pad 25: Ctrl_ALU_Enable -> Ctrl_ALU_Enable_I
- ALU_Low1 pad 28: GND -> Ctrl_ALU_Enable_I
- ALU_Low1 pad 31: VCC -> Ctrl_ALU_Enable_I
- C10 pad 1: GND -> VCC
- C10 pad 2: VCC -> GND
- C11 pad 1: GND -> VCC
- C11 pad 2: VCC -> GND
- Flags1 pad 10: Ctrl_ALU_Enable -> Ctrl_ALU_Enable_I
- Flags1 pad 9: Ctrl_ALU_Enable -> Ctrl_ALU_Enable_I
- Lookup1 pad 19: Net-(Decode_A1-Pad11) -> Ctrl_PC_Count
- Lookup1 pad 20: Net-(Decode_A1-Pad10) -> Ctrl_PC_Input_I
- Lookup1 pad 21: Net-(Decode_A1-Pad9) -> Ctrl_PC_Output_I
- Lookup1 pad 22: Net-(Decode_A1-Pad8) -> Ctrl_ALU_Enable_I
- Lookup1 pad 23: VCC -> GND
- Lookup1 pad 25: VCC -> GND
- Lookup1 pad 31: VCC -> GND
- MAR_A1 pad 10: Ctrl_MAR_Low_Input -> Ctrl_MAR_Low_Input_I
- MAR_A1 pad 11: Data7 -> Data3
- MAR_A1 pad 12: Data6 -> Data2
- MAR_A1 pad 13: Data5 -> Data1
- MAR_A1 pad 14: Data4 -> Data0
- MAR_A1 pad 9: Ctrl_MAR_Low_Input -> Ctrl_MAR_Low_Input_I
- MAR_B1 pad 10: Ctrl_MAR_High_Input -> Ctrl_MAR_Low_Input_I
- MAR_B1 pad 11: Data3 -> Data7
- MAR_B1 pad 12: Data2 -> Data6
- MAR_B1 pad 13: Data1 -> Data5
- MAR_B1 pad 14: Data0 -> Data4
- MAR_B1 pad 9: Ctrl_MAR_High_Input -> Ctrl_MAR_Low_Input_I
- MAR_C1 pad 10: Ctrl_MAR_High_Input -> Ctrl_MAR_High_Input_I
- MAR_C1 pad 11: Data7 -> Data3
- MAR_C1 pad 12: Data6 -> Data2
- MAR_C1 pad 13: Data5 -> Data1
- MAR_C1 pad 14: Data4 -> Data0
- MAR_C1 pad 9: Ctrl_MAR_High_Input -> Ctrl_MAR_High_Input_I
- PC_A1 pad 1: Reset -> Net-(PC_A1-Pad1)
- PC_A1 pad 9: Ctrl_PC_Input -> Ctrl_PC_Input_I
- PC_B1 pad 1: Reset -> Net-(PC_A1-Pad1)
- PC_B1 pad 9: Ctrl_PC_Input -> Ctrl_PC_Input_I
- PC_C1 pad 1: Reset -> Net-(PC_A1-Pad1)
- PC_C1 pad 9: Ctrl_PC_Input -> Ctrl_PC_Input_I
- U1 pad 19: Ctrl_PC_Output -> Ctrl_PC_Output_I
- U2 pad 19: Ctrl_PC_Output -> Ctrl_PC_Output_I
Other:
- net class GND added: clearance 0.2, trace_width 0.5, via_dia 1.2, via_drill 0.8
- net class VCC added: clearance 0.2, trace_width 0.5, via_dia 1.2, via_drill 0.8
- board text added: "AMM812"
- board text added: "AMM812 - October 2018"
- board text added: "Copyright © 2018 Andreas T Jonsson"

Commit message: Updated text.
Parts:
- moved REF1 3.54 mm to (65.0, 65.0)
- moved REF2 3.54 mm to (205.0, 65.0)
- moved REF3 3.54 mm to (205.0, 155.0)
- moved REF4 3.54 mm to (65.0, 155.0)
Other:
- board text added: "AMM816"
- board text removed: "AMM812"
Changed lines of the file:
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@@
     (descr "16-lead dip package, row spacing 7.62 mm (300 mils)")
     (tags "dil dip 2.54 300")
-    (fp_text reference PC_C1 (at 0 -5.22 90) (layer F.SilkS)
+    (fp_text reference PC_C1 (at 2.5 -5 90) (layer F.SilkS)
       (effects (font (size 1 1) (thickness 0.15)))
     )
@@
     (descr "20-lead dip package, row spacing 7.62 mm (300 mils)")
     (tags "dil dip 2.54 300")
-    (fp_text reference U2 (at 10 5 180) (layer F.SilkS)
+    (fp_text reference U2 (at 10 10 180) (layer F.SilkS)
       (effects (font (size 1 1) (thickness 0.15)))
     )
@@
     (descr "20-lead dip package, row spacing 7.62 mm (300 mils)")
     (tags "dil dip 2.54 300")
-    (fp_text reference U4 (at 0 -5.22) (layer F.SilkS)
+    (fp_text reference U4 (at 2.5 -5) (layer F.SilkS)
       (effects (font (size 1 1) (thickness 0.15)))
     )
@@
   )
   (module Connect:1pin (layer F.Cu)
-    (at 67.5 67.5)
+    (at 65 65)
     (descr "module 1 pin (ou trou mecanique de percage)")
     (tags DEV)
@@
   )
   (module Connect:1pin (layer F.Cu)
-    (at 202.5 67.5)
+    (at 205 65)
     (descr "module 1 pin (ou trou mecanique de percage)")
     (tags DEV)
@@
   )
   (module Connect:1pin (layer F.Cu)
-    (at 202.5 152.5)
+    (at 205 155)
     (descr "module 1 pin (ou trou mecanique de percage)")
     (tags DEV)
@@
   )
   (module Connect:1pin (layer F.Cu)
-    (at 67.5 152.5)
+    (at 65 155)
     (descr "module 1 pin (ou trou mecanique de percage)")
     (tags DEV)
@@
     (effects (font (size 1 1) (thickness 0.2)))
   )
-  (gr_text AMM812 (at 115 127.5) (layer F.SilkS)
+  (gr_text AMM816 (at 115 127.5) (layer F.SilkS)
     (effects (font (size 4 4) (thickness 0.7)))
   )

Commit message: Just a backup.
Parts:
- moved U3 21.4 mm to (67.5, 147.5), turned to 90 degrees
- moved C13 20.2 mm to (87.5, 145.0), turned to 90 degrees
- moved C2 2.50 mm to (117.5, 120.0)
- moved C32 2.50 mm to (195.0, 122.5)
- moved IR_High1 2.50 mm to (112.5, 97.5)
Other:
- board text added: "AMM816 - October 2018"
- board text added: "https://gitlab.com/phix/amm816"
- board text removed: "AMM812 - October 2018"
